Commit message: Update robot_core.xacro

File: description/robot_core.xacro (robot description, xacro)
@@ -44,4 +44,9 @@
         </xacro:inertial_box>
     </link>
+    <gazebo reference="chassis">
+        <material>
+            Gazebo/Black
+        </material>
+    </gazebo>
     <!-- LEFT WHEEL LINK -->
     <joint name="left_wheel_joint" type="continuous">
@@ -67,4 +72,9 @@
         </xacro:inertial_cylinder>
     </link>
+    <gazebo reference="left_wheel">
+        <material>
+            Gazebo/Green
+        </material>
+    </gazebo>
     <!-- RIGHT WHEEL LINK -->
     <joint name="right_wheel_joint" type="continuous">
@@ -90,4 +100,9 @@
         </xacro:inertial_cylinder>
     </link>
+    <gazebo reference="right_wheel">
+        <material>
+            Gazebo/Green
+        </material>
+    </gazebo>
     <!-- CASTER WHEEL LINK -->
     <joint name="caster_wheel_joint" type="fixed">
@@ -112,3 +127,8 @@
         </xacro:inertial_sphere>
     </link>
+    <gazebo reference="caster_wheel">
+        <material>
+            Gazebo/White
+        </material>
+    </gazebo>
 </robot>
